File: PCB/bugboard.kicad_sch (KiCad schematic)
At the start: 27 parts, among them J1 USB_C_Receptacle_USB2.0_16P, J2 Conn_01x04, J3 Conn_01x20, J4 Conn_01x20, SW1 SW_SPST, SW2 SW_SPST, U1 STM32G431CBTx, U2 XC6206PxxxMR

Commit message: Added PCB and Schematic
Parts:
- SW1, SW2: footprint Button_Switch_SMD:SW_SPST_EVPBF -> Button_Switch_SMD:SW_SPST_TS-1088-xR020
